Commit message: Fix rotation of map cloud

File: urdf/udacity_bot.xacro (robot description, xacro)
@@ -25,5 +25,5 @@
   </joint>
   <joint type="fixed" name="camera_joint">
-    <origin xyz="0.2 0 0" rpy="0 0 0"/>
+    <origin xyz="0.4 0 0" rpy="0 0 0"/>
     <child link="camera"/>
     <parent link="chassis"/>
@@ -51,4 +51,11 @@
       </geometry>
     </visual>
+  </link>
+  <joint type="fixed" name="camera_optical_joint">
+    <origin xyz="0 0 0" rpy="-1.57 0 -1.57"/>
+    <child link="camera_optical"/>
+    <parent link="camera"/>
+  </joint>
+  <link name="camera_optical">
   </link>
   <joint type="fixed" name="hokuyo_joint">
